File: Electrical/MicrocontrollerInputModule/MicrocontrollerInputModule.kicad_pro.kicad_sch (KiCad schematic)
At the start: 46 parts, among them J1 Conn_02x04_Odd_Even, J2 Conn_01x16, J3 Conn_01x10, SW1 KXT3, SW2 KXT3, U1 W25Q16JVUXIQ, U2 RP2040, Y1 12.000MHz

Commit message: Rename to Microcontroller Input Module
Other:
- title: Minimal Input Module Reference Design -> Microcontroller Input Module
